File: pcb/_autosave-babycall-pcb.kicad_sch (KiCad schematic)
At the start: 35 parts, among them SW1 TS-1187A-B-A-B, SW2 TS-1187A-B-A-B, U1 ESP32-C3-MINI-1-H4X, U2 BQ24074RGTR, U3 AP2112K-3.3, U4 ICS-43434_C5656610

Commit message: Working on schematic
Parts:
- removed C4: 1uF, PCM_JLCPCB:C_0402, symbol PCM_JLCPCB-Capacitors:0402,1uF
- removed C5, C6: 4.7uF, PCM_JLCPCB:C_0402, symbol PCM_JLCPCB-Capacitors:0402,4.7uF
- removed R2, R3, R4: 10kΩ, PCM_JLCPCB:R_0402, symbol PCM_JLCPCB-Resistors:0402,10kΩ
- removed R5, R9: 3kΩ, PCM_JLCPCB:R_0603, symbol PCM_JLCPCB-Resistors:0603,3kΩ
- removed U2: BQ24074RGTR, jlcpcb:QFN-16_L3.0-W3.0-P0.50-TL-EP1.7, symbol JLCPCB:BQ24074RGTR
- added C9: 1uF, PCM_JLCPCB:C_0402, symbol PCM_JLCPCB-Capacitors:0402,1uF
- added D5: Red, PCM_JLCPCB:D_0603, symbol PCM_JLCPCB-Diodes:LED,0603,Red
- added D6, D7: SS34, PCM_JLCPCB:D_SMA, symbol PCM_JLCPCB-Diodes:Schottky,SS34,(2)
- added R14: 330Ω, PCM_JLCPCB:R_0402, symbol PCM_JLCPCB-Resistors:0402,330Ω
- added R15: 2kΩ, PCM_JLCPCB:R_0402, symbol PCM_JLCPCB-Resistors:0402,2kΩ
- added U5: TP4054, PCM_JLCPCB:SOT-23-5_L3.0-W1.7-P0.95-LS2.8-BL, symbol PCM_JLCPCB-Power:Battery, Li-Ion, 0.8A, TP4054
Connections:
- net +5V: now also C9.2, D6.2, R14.2, U5.4 (VCC)
- net +BATT: now also D7.2, U5.3 (BAT)
- net GND: now also C9.1, R15.1, U5.2 (GND)
- net +4.4V: no longer names the net of C10.2, U3.1 (VIN), U3.3 (EN)
- net +4.4V: now also D6.1, D7.1
- net CHG: no longer names the net of U1.18 (IO4)
- net PGOOD: no longer names the net of U1.19 (IO5)
- new net: D5.2, R14.1
- new net: D5.1, U5.1 (CHRG)
- new net: R15.2, U5.5 (PROG)
Other:
- note added: "300mA"
- note added: "Regulator"
- note added: "Revisit this, make sure pins are correct"
- note removed: "LDO"
- note removed: "Thermal pad should be connected to GND"
- moved on the sheet: C10, C11, C7, C8, R7, R8, U3, USB1
